File: ultimateFC.kicad_pcb (KiCad board)
At the start: 6 copper layers, 36 x 36 mm, 205 parts, among them J1 USB_B_Micro, U1 LMR33630CQRNX, U2 TPS62824ADMQ, U3 LMR33620CRNXT, U4 S25FL064L, U5 DPS310, U6 BMI270, U7 STM32H735VGH6, U8 ICM-20602, Y1 CSTNE8M00G550000R0

Commit message: more layout
Parts:
- TP101, TP60: moved to B.Cu
- moved TP60 52.7 mm to (111.1, 110.9), turned to 180 degrees
- moved TP101 51.4 mm to (113.1, 106.9), turned to 180 degrees
- moved TP59 44.5 mm to (111.1, 106.9)
- moved R17 8.15 mm to (103.9, 102.8)
- moved R16 7.76 mm to (105.8, 103.0)
- moved U6 6.71 mm to (105.2, 106.9)
- moved R15 6.67 mm to (102.8, 104.4)
- moved C35 4.96 mm to (104.0, 119.5)
- moved U8 4.96 mm to (104.9, 117.3)
- moved R14 4.49 mm to (102.8, 106.4)
- moved L4 3.80 mm to (115.4, 114.8)
- moved TP10 2.79 mm to (118.2, 106.5)
- moved TP44 2.79 mm to (118.2, 108.5)
- moved TP11 2.79 mm to (116.0, 106.5)
- moved TP43 2.79 mm to (116.0, 108.5)
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Connections:
- net UC_LED_2 renamed IMU_INT1A
- TP60 pad 1: Net-(TP60-Pad1) -> IMU_INT1B
- U7 pad A4: Net-(U7-PadA4) -> Net-(TP41-Pad1)
- U7 pad A6: Net-(U7-PadA6) -> Net-(TP38-Pad1)
- U7 pad A8: Net-(U7-PadA8) -> Net-(TP52-Pad1)
- U7 pad B1: Net-(U7-PadB1) -> Net-(TP85-Pad1)
- U7 pad B2: Net-(U7-PadB2) -> Net-(TP102-Pad1)
- U7 pad B3: Net-(U7-PadB3) -> Net-(TP94-Pad1)
- U7 pad B6: Net-(U7-PadB6) -> Net-(TP36-Pad1)
- U7 pad B7: Net-(U7-PadB7) -> Net-(TP53-Pad1)
- U7 pad B8: Net-(U7-PadB8) -> Net-(TP50-Pad1)
- U7 pad C5: Net-(U7-PadC5) -> Net-(TP37-Pad1)
- U7 pad C6: Net-(U7-PadC6) -> Net-(TP56-Pad1)
- U7 pad C7: Net-(U7-PadC7) -> Net-(TP49-Pad1)
- U7 pad E10: Net-(U7-PadE10) -> Net-(TP87-Pad1)
- U7 pad E3: Net-(U7-PadE3) -> Net-(TP42-Pad1)
- U7 pad E4: Net-(U7-PadE4) -> Net-(TP84-Pad1)
- U7 pad E9: Net-(R26-Pad2) -> /USB_VBUS_sense
- U7 pad F1: Net-(U7-PadF1) -> Net-(TP72-Pad1)
- U7 pad F10: Net-(U7-PadF10) -> Net-(TP86-Pad1)
- U7 pad F3: Net-(U7-PadF3) -> Net-(TP71-Pad1)
- U7 pad F4: Net-(U7-PadF4) -> Net-(TP73-Pad1)
- U7 pad G4: Net-(U7-PadG4) -> Net-(TP74-Pad1)
- U7 pad H4: Net-(U7-PadH4) -> Net-(TP75-Pad1)
- U7 pad H6: Net-(U7-PadH6) -> Net-(TP101-Pad1)
- U7 pad H7: Net-(U7-PadH7) -> IMU_INT1B
- U7 pad J5: Net-(U7-PadJ5) -> Net-(TP35-Pad1)
- U7 pad K1: Net-(U7-PadK1) -> Net-(TP107-Pad1)
- U7 pad K6: Net-(U7-PadK6) -> Net-(TP100-Pad1)
Routing:
- net Net-(J1-Pad3): track 11.4 -> 0.00 mm, vias 0 -> 1
- net Net-(J1-Pad2): track 10.5 -> 0.00 mm, vias 0 -> 1
- net MISO_OSD: track 0.00 -> 8.84 mm, vias 0 -> 1
- net SCLK_OSD: track 0.00 -> 8.13 mm, vias 0 -> 1
- net IMU_INT1A: track 0.00 -> 7.24 mm, vias 0 -> 1
- net Net-(R12-Pad2): track 6.97 -> 0.00 mm
- net Net-(TP101-Pad1): track 0.00 -> 6.96 mm, vias 0 -> 1
- net CS_OSD: track 0.00 -> 6.09 mm
- net Net-(R20-Pad2): track 0.00 -> 5.11 mm
- net Net-(R13-Pad2): track 4.71 -> 0.00 mm
- net Net-(R16-Pad2): track 4.46 -> 0.00 mm
- net MOSI_OSD: track 0.00 -> 4.38 mm
- net Net-(R19-Pad2): track 0.00 -> 4.24 mm
- net IMU_INT1B: track 0.00 -> 4.21 mm, vias 0 -> 1
- net Net-(R14-Pad2): track 3.29 -> 0.00 mm
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
Commit message: update layout
Parts:
- moved D4 93.8 mm to (103.8, 115.2), turned to -90 degrees
- moved TP100 79.8 mm to (106.5, 83.4)
- moved TP75 32.0 mm to (106.2, 101.0)
- moved TP73 31.4 mm to (108.2, 101.0)
- moved TP12 25.8 mm to (119.0, 118.4)
- moved TP93 24.1 mm to (119.0, 120.4)
- moved U4 23.9 mm to (118.9, 122.0), turned to 90 degrees
- moved TP18 23.1 mm to (121.2, 118.4)
- moved TP97 23.1 mm to (121.2, 120.4)
- moved TP19 23.1 mm to (121.2, 125.0)
- moved TP96 23.1 mm to (121.2, 123.0)
- moved TP95 22.8 mm to (119.0, 123.0)
- moved TP13 22.5 mm to (119.0, 125.0)
- moved TP102 18.0 mm to (146.9, 93.4)
- moved TP85 18.0 mm to (146.9, 90.9)
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Routing:
- net CS_OSD: track 6.09 -> 21.6 mm, vias 0 -> 1
- net Net-(C36-Pad1): track 4.19 -> 16.5 mm, vias 0 -> 2
- net MOSI_OSD: track 4.38 -> 16.4 mm, vias 0 -> 1
- net Net-(J1-Pad3): track 0.00 -> 11.7 mm, vias 1 -> 0
- net UART9_RX: track 0.00 -> 11.7 mm, vias 0 -> 1
- net +3V3: track 6.09 -> 17.5 mm, vias 10 -> 14
- net MP_PIN2: track 0.00 -> 10.9 mm, vias 0 -> 1
- net Net-(J1-Pad2): track 0.00 -> 10.7 mm, vias 1 -> 0
- net UART9_TX: track 0.00 -> 10.4 mm, vias 0 -> 1
- net Net-(TP73-Pad1): track 0.00 -> 9.96 mm, vias 0 -> 1
- net UART7_RX: track 0.00 -> 9.95 mm, vias 0 -> 1
- net CS_FLASH: track 0.00 -> 8.90 mm, vias 0 -> 1
- net UART4_TX: track 0.00 -> 8.75 mm, vias 0 -> 1
- net MOTOR1: track 0.00 -> 8.65 mm, vias 0 -> 1
- net I2C_SDA: track 0.00 -> 8.63 mm, vias 0 -> 1
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- added copper zone on In2.Cu, net +3V3
- added copper zone on In3.Cu, net +5V
- added copper zone on In1.Cu, net GND
- added copper zone on In4.Cu, net GND

Commit message: layout update
Parts:
- TP103, TP106, TP37, TP39, TP49, TP56, TP57, TP58, TP63, TP64, TP73, TP74, TP75, TP84, TP91, TP92, TP98: moved to B.Cu
- TP51: moved to F.Cu
- moved TP9 101.6 mm to (163.7, 102.4)
- moved TP74 85.3 mm to (121.9, 88.7), turned to 180 degrees
- moved TP84 84.4 mm to (138.1, 98.0), turned to 180 degrees
- moved TP91 83.7 mm to (129.1, 123.5), turned to -90 degrees
- moved TP106 76.5 mm to (114.0, 93.7), turned to 180 degrees
- moved TP34 75.4 mm to (128.1, 92.5)
- moved TP28 74.4 mm to (112.2, 136.0)
- moved TP64 73.7 mm to (112.2, 100.8), turned to 180 degrees
- moved TP92 71.1 mm to (129.1, 121.3), turned to -90 degrees
- moved TP98 70.3 mm to (117.4, 91.5), turned to 180 degrees
- moved TP99 68.3 mm to (117.6, 88.9)
- moved TP39 67.1 mm to (115.0, 142.5), turned to 180 degrees
- moved TP36 65.7 mm to (111.3, 140.7)
- moved R22 64.7 mm to (120.7, 116.5)
- moved TP35 61.9 mm to (130.3, 89.7)
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Connections:
- net Net-(R22-Pad2) renamed /NRST
Routing:
- net MOTOR3: track 2.94 -> 24.8 mm, vias 0 -> 1
- net MOTOR4: track 3.86 -> 25.7 mm, vias 0 -> 1
- net MOTOR2: track 3.88 -> 22.6 mm, vias 0 -> 1
- net MOTOR1: track 8.65 -> 26.3 mm, vias 1 -> 3
- net CS_GYRO: track 4.31 -> 21.9 mm, vias 0 -> 1
- net MISO_GYRO: track 3.09 -> 19.7 mm, vias 0 -> 1
- net MOSI_GYRO: track 4.31 -> 18.4 mm, vias 0 -> 1
- net SCLK_GYRO: track 9.41 -> 19.9 mm, vias 0 -> 1
- net UART3_RX: track 0.42 -> 10.7 mm
- net Net-(C36-Pad1): track 16.5 -> 9.93 mm
- net /USB_VBUS_sense: track 4.68 -> 11.1 mm
- net +3V3: track 17.5 -> 11.4 mm
- net USB_VBUS: track 0.00 -> 5.40 mm
- net Net-(TP87-Pad1): track 2.87 -> 5.84 mm, vias 0 -> 1
- net UART8_RX: track 2.51 -> 5.47 mm, vias 0 -> 1
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Other:
- board text removed: "If you want to (commercially) manufacture this, we strongly recommend to contact us before ( yolofc@weber-ee.de )."
- board text removed: "Please use the correct layer stackup, via in pad and sideplating options."
- board text removed: "Sideplating"
- board text removed: "When using this commercially, please be fair and mention our names ( crteensy / chris_fly ) on some prominet place"
