File: ultimateFC.kicad_pcb (KiCad board)
At the start: 6 copper layers, 36 x 36 mm, 205 parts, among them J1 USB_B_Micro, U1 LMR33630CQRNX, U2 TPS62824ADMQ, U3 LMR33620CRNXT, U4 S25FL064L, U5 DPS310, U6 BMI270, U7 STM32H735VGH6, U8 ICM-20602, Y1 CSTNE8M00G550000R0

Commit message: update layout
Parts:
- TP39, TP57, TP58: moved to F.Cu
- TP76, TP9: moved to B.Cu
- moved TP9 40.8 mm to (124.8, 114.9)
- moved R6 40.2 mm to (125.8, 114.6)
- moved C25 39.8 mm to (125.8, 113.6)
- moved R5 38.6 mm to (125.8, 115.6), turned to 180 degrees
- moved TP37 22.8 mm to (113.9, 126.7), turned to 180 degrees
- moved TP56 20.5 mm to (111.9, 126.7), turned to 180 degrees
- moved TP52 18.9 mm to (113.2, 126.7)
- moved TP49 18.1 mm to (109.9, 126.7), turned to 180 degrees
- moved TP53 18.0 mm to (114.3, 129.2)
- moved TP36 14.6 mm to (115.4, 126.7)
- moved TP57 14.1 mm to (100.9, 125.3), turned to -90 degrees
- moved TP40 14.0 mm to (117.6, 126.7)
- moved TP39 13.8 mm to (118.7, 129.2), turned to 0 degrees
- moved TP41 13.5 mm to (119.8, 126.7)
- moved TP50 13.3 mm to (110.1, 127.4)
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Routing:
- net /SWDCLK: track 4.76 -> 17.1 mm
- net /SWDIO: track 4.33 -> 15.4 mm
- net UART3_TX: track 4.03 -> 8.62 mm, vias 1 -> 2
- net UART3_RX: track 10.7 -> 12.8 mm

Commit message: update layout
Parts:
- added REF**: PinHeader_1x05_P2.54mm_Vertical, Connector_PinHeader_2.54mm:PinHeader_1x05_P2.54mm_Vertical, F.Cu at (104.0, 134.2)
- TP36, TP38, TP39, TP40, TP41, TP52, TP53, TP86, TP87, TP94: moved to B.Cu
- moved D2 101.1 mm to (98.5, 123.6)
- moved D3 100.6 mm to (98.5, 124.8)
- moved R24 100.0 mm to (100.4, 123.6), turned to 180 degrees
- moved R25 98.3 mm to (100.4, 124.8), turned to 180 degrees
- moved TP69 41.9 mm to (100.3, 123.1)
- moved TP70 39.2 mm to (100.3, 125.3)
- moved TP62 18.2 mm to (107.8, 123.5)
- moved TP61 16.0 mm to (106.6, 123.6)
- moved TP55 13.1 mm to (118.9, 129.0)
- moved TP54 13.1 mm to (116.7, 129.0)
- moved TP86 9.00 mm to (98.3, 125.3), turned to 90 degrees
- moved TP87 5.87 mm to (98.3, 123.1), turned to 90 degrees
- moved TP57 2.40 mm to (103.3, 125.2)
- moved TP58 2.40 mm to (103.3, 123.0)
- moved TP41 2.31 mm to (120.0, 129.0), turned to 180 degrees
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Connections:
- net Net-(TP86-Pad1) renamed UC_LED_2
- TP51 pad 1: UC_LED_1 -> Net-(TP51-Pad1)
- TP87 pad 1: Net-(TP87-Pad1) -> UC_LED_1
- U7 pad A9: UC_LED_1 -> Net-(TP51-Pad1)
- U7 pad E10: Net-(TP87-Pad1) -> UC_LED_1
Routing:
- net UC_LED_1: track 1.93 -> 18.5 mm, vias 0 -> 1
- net UC_LED_2: track 5.08 -> 20.3 mm
- net UART2_RX: track 1.40 -> 13.2 mm
- net UART2_TX: track 6.88 -> 18.4 mm, vias 1 -> 2
- net Net-(TP94-Pad1): track 3.50 -> 14.7 mm, vias 0 -> 1
- net MP_PIN5: track 4.01 -> 14.9 mm, vias 0 -> 1
- net Net-(TP41-Pad1): track 2.25 -> 12.5 mm, vias 0 -> 1
- net Net-(TP87-Pad1): track 5.84 -> 0.00 mm, vias 1 -> 0
- net Net-(C23-Pad2): track 0.98 -> 5.36 mm, vias 1 -> 2
- net MOTOR1: track 26.3 -> 23.3 mm
- net UART3_TX: track 8.62 -> 11.0 mm
- net Net-(TP51-Pad1): track 0.00 -> 1.93 mm
- net UART3_RX: track 12.8 -> 14.6 mm, vias 1 -> 2
- net Net-(R11-Pad1): track 1.40 -> 2.67 mm
- net MP_PIN6: track 2.37 -> 3.59 mm
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
Commit message: add WS2812, update layout
Parts:
- removed REF**: PinHeader_1x05_P2.54mm_Vertical, Connector_PinHeader_2.54mm:PinHeader_1x05_P2.54mm_Vertical
- added D5: WS2812B, LED_SMD:LED_WS2812B_PLCC4_5.0x5.0mm_P3.2mm, F.Cu at (102.8, 124.2)
- added D6: SBR1A30T5-7, Diode_SMD:D_SOD-523, F.Cu at (107.0, 125.3)
- added SW1: SW_Push, Button_Switch_SMD:SW_Push_1P1T_NO_CK_KMR2, F.Cu at (105.9, 128.7)
- added TP112: Pad, TestPoint:TestPoint_Pad_1.5x1.5mm, F.Cu at (131.7, 121.0)
- added TP113: Pad, TestPoint:TestPoint_Pad_1.5x1.5mm, F.Cu at (131.7, 125.4)
- added TP114: Pad, TestPoint:TestPoint_Pad_1.5x1.5mm, B.Cu at (102.8, 123.1)
- added TP115: Pad, TestPoint:TestPoint_Pad_1.5x1.5mm, F.Cu at (111.2, 126.3)
- added TP116: Pad, TestPoint:TestPoint_Pad_1.5x1.5mm, F.Cu at (112.3, 129.0)
- TP102, TP105, TP107, TP109, TP15, TP42, TP50, TP51, TP61, TP62, TP71, TP72, TP85: moved to B.Cu
- TP103, TP98: moved to F.Cu
- TP28: value bridge -> Pad; footprint ultimateFC:solderbridge_tiny -> TestPoint:TestPoint_Pad_1.5x1.5mm
- moved TP6 34.6 mm to (110.1, 129.0), turned to 180 degrees
- moved TP71 29.4 mm to (121.8, 103.7), turned to 180 degrees
- moved TP42 26.4 mm to (124.0, 103.7), turned to 180 degrees
- moved TP105 23.6 mm to (122.9, 101.0), turned to 180 degrees
- moved TP107 23.2 mm to (120.7, 101.0), turned to 180 degrees
- moved TP72 22.5 mm to (125.1, 101.0), turned to 180 degrees
- moved TP17 18.2 mm to (131.7, 123.2), turned to 90 degrees
- moved TP84 17.7 mm to (128.2, 112.7), turned to -90 degrees
- moved TP109 16.5 mm to (118.5, 101.0), turned to 180 degrees
- moved TP58 14.7 mm to (116.7, 129.0), turned to 0 degrees
- moved TP104 14.0 mm to (120.7, 101.0)
- moved TP100 13.1 mm to (117.4, 103.7)
- moved TP34 12.6 mm to (119.6, 103.7)
- moved TP35 12.5 mm to (121.8, 103.7)
- moved TP99 12.5 mm to (118.5, 101.0)
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Connections:
- TP28 pad 1: +3V3 -> +5V
Routing:
- net Net-(R11-Pad1): track 2.67 -> 32.1 mm, vias 0 -> 2
- net /NRST: track 4.20 -> 29.8 mm, vias 0 -> 2
- net Net-(TP50-Pad1): track 2.84 -> 20.9 mm, vias 0 -> 1
- net UART3_RX: track 14.6 -> 31.4 mm
- net curr_sig: track 2.23 -> 18.1 mm, vias 0 -> 2
- net Net-(TP72-Pad1): track 4.11 -> 19.9 mm, vias 0 -> 1
- net MP_PIN3: track 3.13 -> 18.8 mm, vias 0 -> 1
- net ESC_4_TX: track 3.79 -> 18.9 mm
- net Net-(TP107-Pad1): track 1.07 -> 15.7 mm, vias 0 -> 1
- net ESC_2_TX: track 3.72 -> 18.2 mm, vias 0 -> 1
- net Net-(TP102-Pad1): track 3.91 -> 17.9 mm, vias 0 -> 1
- net ESC_1_TX: track 3.28 -> 17.0 mm
- net UART8_RX: track 5.47 -> 19.2 mm
- net Net-(TP42-Pad1): track 3.57 -> 17.3 mm
- net vol_sig: track 5.06 -> 18.0 mm, vias 0 -> 3
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
Commit message: MORE PADS!!!
Parts:
- added TP117: Pad, TestPoint:TestPoint_Pad_1.5x1.5mm, B.Cu at (111.4, 116.2)
- added TP118: Pad, TestPoint:TestPoint_Pad_1.5x1.5mm, B.Cu at (101.0, 117.6)
- added TP119: Pad, TestPoint:TestPoint_Pad_1.5x1.5mm, B.Cu at (98.2, 116.5)
- added TP120: Pad, TestPoint:TestPoint_Pad_1.5x1.5mm, B.Cu at (98.2, 118.7)
- added TP121: Pad, TestPoint:TestPoint_Pad_1.5x1.5mm, F.Cu at (121.8, 98.3)
- added TP122: Pad, TestPoint:TestPoint_Pad_1.5x1.5mm, B.Cu at (121.8, 98.3)
- added TP123: Pad, TestPoint:TestPoint_Pad_1.5x1.5mm, B.Cu at (108.6, 98.3)
- added TP124: Pad, TestPoint:TestPoint_Pad_1.5x1.5mm, B.Cu at (106.4, 98.3)
- added TP125: Pad, TestPoint:TestPoint_Pad_1.5x1.5mm, F.Cu at (119.6, 98.3)
- added TP126: Pad, TestPoint:TestPoint_Pad_1.5x1.5mm, F.Cu at (124.0, 98.3)
- added TP127: Pad, TestPoint:TestPoint_Pad_1.5x1.5mm, B.Cu at (110.8, 98.3)
- added TP128: Pad, TestPoint:TestPoint_Pad_1.5x1.5mm, B.Cu at (119.6, 98.3)
- added TP129: Pad, TestPoint:TestPoint_Pad_1.5x1.5mm, B.Cu at (117.4, 98.3)
- added TP130: Pad, TestPoint:TestPoint_Pad_1.5x1.5mm, B.Cu at (124.0, 98.3)
- added TP131: Pad, TestPoint:TestPoint_Pad_1.5x1.5mm, B.Cu at (115.2, 98.3)
- added TP132: Pad, TestPoint:TestPoint_Pad_1.5x1.5mm, B.Cu at (113.0, 98.3)
- added TP133: Pad, TestPoint:TestPoint_Pad_1.5x1.5mm, B.Cu at (104.2, 98.3)
- added TP134: Pad, TestPoint:TestPoint_Pad_1.5x1.5mm, F.Cu at (131.7, 123.2)
- added TP135: Pad, TestPoint:TestPoint_Pad_1.5x1.5mm, F.Cu at (131.7, 125.4)
- added TP136: Pad, TestPoint:TestPoint_Pad_1.5x1.5mm, F.Cu at (131.7, 120.8)
- added TP137: Pad, TestPoint:TestPoint_Pad_1.5x1.5mm, B.Cu at (111.9, 131.7)
- added TP138: Pad, TestPoint:TestPoint_Pad_1.5x1.5mm, B.Cu at (106.7, 131.7)
- added TP139: Pad, TestPoint:TestPoint_Pad_1.5x1.5mm, B.Cu at (114.4, 131.7)
- added TP140: Pad, TestPoint:TestPoint_Pad_1.5x1.5mm, B.Cu at (109.3, 131.7)
- added TP141: Pad, TestPoint:TestPoint_Pad_1.5x1.5mm, B.Cu at (104.2, 131.7)
- added TP142: Pad, TestPoint:TestPoint_Pad_1.5x1.5mm, B.Cu at (117.8, 131.7)
- added TP143: Pad, TestPoint:TestPoint_Pad_1.5x1.5mm, B.Cu at (120.0, 131.7)
- moved TP5 10.3 mm to (115.2, 98.3)
- moved TP4 8.80 mm to (117.4, 98.3)
- moved TP2 6.60 mm to (113.0, 98.3)
- moved TP7 6.60 mm to (106.4, 98.3)
- moved TP8 4.40 mm to (110.8, 98.3)
- moved TP3 2.20 mm to (108.6, 98.3)
- moved C38 0.10 mm to (114.4, 114.7)
Connections:
- net /SWDCLK renamed SWDCLK
- net /SWDIO renamed SWDIO
Routing:
- net Net-(J1-Pad3): track 11.7 -> 15.4 mm, vias 0 -> 1
- net Net-(J1-Pad2): track 10.7 -> 13.7 mm, vias 0 -> 1
- net SWDIO: track 26.0 -> 23.5 mm
- net USB_VBUS: track 5.40 -> 7.73 mm, vias 0 -> 1
- net +3V3: track 18.7 -> 20.1 mm, vias 15 -> 16
- net SWDCLK: track 22.6 -> 21.8 mm
- net /USB_VBUS_sense: vias 0 -> 1

Commit message: DCDC layouts
Parts:
- moved C21 52.4 mm to (141.5, 115.2)
- moved C20 49.2 mm to (147.5, 112.1)
- moved C19 45.2 mm to (147.5, 109.6)
- moved C8 43.8 mm to (142.5, 111.8)
- moved C22 42.0 mm to (148.3, 106.8)
- moved C18 40.1 mm to (153.2, 106.5)
- moved C7 38.8 mm to (142.5, 107.4)
- moved C9 34.3 mm to (147.8, 114.4)
- moved C13 32.6 mm to (144.9, 114.9)
- moved C16 31.9 mm to (150.9, 113.3)
- moved C14 29.3 mm to (150.9, 109.4)
- moved C12 27.0 mm to (153.8, 108.7)
- moved C17 26.7 mm to (150.9, 111.3)
- moved C10 24.6 mm to (153.8, 110.7)
- moved C15 18.6 mm to (156.6, 106.2)
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Connections:
- R11 pad 1: Net-(U7-PadA5) -> Net-(R11-Pad1)
- SW1 pad 1: Net-(U7-PadA5) -> Net-(R11-Pad1)
Routing:
- net Net-(U7-PadA5): track 32.1 -> 0.00 mm, vias 2 -> 0
- net Net-(R11-Pad1): track 0.00 -> 32.1 mm, vias 0 -> 2
- net +BATT: track 0.00 -> 6.95 mm
- net Net-(C30-Pad1): track 0.00 -> 3.65 mm
- net Net-(R10-Pad1): track 2.95 -> 6.30 mm, vias 1 -> 2
- net Net-(D1-Pad1): track 0.00 -> 3.23 mm
- net Net-(C5-Pad1): track 7.73 -> 5.49 mm, vias 0 -> 2
- net GND: track 21.7 -> 19.6 mm, vias 51 -> 57
- net Net-(C25-Pad1): track 0.00 -> 2.01 mm, vias 0 -> 1
- net Net-(C3-Pad1): track 0.00 -> 1.92 mm
- net Net-(R1-Pad2): track 0.50 -> 2.19 mm
- net +10V: track 0.00 -> 1.61 mm
- net Net-(C29-Pad1): track 0.00 -> 1.00 mm
- net Net-(C11-Pad1): track 0.97 -> 1.96 mm
- net Net-(C30-Pad2): track 0.00 -> 0.98 mm
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- added copper zone on F.Cu, net +10V
- added copper zone on F.Cu, net Net-(C1-Pad1)
- added copper zone on F.Cu, net Net-(C27-Pad1)
- added copper zone on F.Cu, net Net-(C30-Pad1)
- added copper zone on F.Cu, net Net-(C31-Pad1)
- removed copper zone on F.Cu, net Net-(C35-Pad1)

Commit message: layout tweaks
Parts:
- moved L4 0.15 mm to (117.2, 116.2)
- turned Y1 to 90 degrees
Connections:
- U7 pad A5: Net-(U7-PadA5) -> Net-(R11-Pad1)
Routing:
- net Net-(U7-PadG1): track 2.81 -> 3.47 mm
- net GND: track 19.6 -> 19.5 mm, vias 57 -> 54
